File: Eagle/DCCShield.brd (EAGLE design)
At the start: 59.7 x 53.3 mm, 7 parts

Commit message: Updated to ver 1.1
Parts:
- added ACK: (no value), pinhead:1X01
- added B2: (no value), rectifier:RB1A
- added OK2: PC817, optocoupler:DIL04
- added Q1: BC557, transistor-pnp:TO92
- added R3: 1k, rcl:0207/10
- added R4: 100, rcl:0207/10
- moved OK1 8.25 mm to (45.7, 38.7)
- moved PIN 5.46 mm to (15.9, 38.7)
- moved R2 4.58 mm to (39.4, 20.3)
- moved D1 4.07 mm to (40.0, 11.4)
- moved R1 4.07 mm to (39.4, 15.9)
Connections:
- removed net N$3: D1.A, DCC.2, OK1.3
- new net DCC_1: B2.AC1, DCC.1, R1.1
- new net DCC_2: B2.AC2, D1.A, DCC.2, OK1.3
- new net N$10: Q1.1, R4.1
- new net N$11: B2.+, R4.2
- new net N$4: ACK.1, R3.1
- new net N$8: OK2.1, R3.2
- new net N$9: OK2.4, Q1.2
- net GND: now also OK2.2
- net N$1: now also B2.-, OK2.3, Q1.3; no longer DCC.1, R1.1
Routing:
- net DCC_2: track 0.00 -> 65.1 mm
- net N$8: track 0.00 -> 43.6 mm
- net DCC_1: track 0.00 -> 36.5 mm
- net N$11: track 0.00 -> 32.4 mm
- net N$3: track 31.6 -> 0.00 mm
- net N$4: track 0.00 -> 21.9 mm
- net N$9: track 0.00 -> 21.6 mm
- net N$5: track 36.9 -> 56.0 mm
- net GND: track 75.4 -> 91.8 mm
- net N$10: track 0.00 -> 13.8 mm
- net N$1: track 24.0 -> 35.0 mm
- net +5V: track 38.9 -> 49.3 mm
- net N$6: track 39.9 -> 44.5 mm
- net N$7: track 31.9 -> 35.1 mm
- net N$2: track 32.1 -> 31.5 mm
Other:
- board text added: "ACK PIN"
- board text added: "DCC IN"
- board text added: "DCC PIN"
- board text added: "PdL DCCShield v1.1"
- board text removed: "PdL DCCShield v1.0"
