File: Eagle/DCCShield.sch (EAGLE design)
At the start: 7 parts

Commit message: Updated to ver 1.1
Parts:
- added ACK: (no value), pinhead:PINHD-1X1
- added B2: (no value), rectifier:RB1A
- added OK2: PC817, optocoupler:PC817
- added Q1: BC557, transistor-pnp:BC557
- added R3: 1k, rcl:R-EU_0207/10
- added R4: 100, rcl:R-EU_0207/10
Connections:
- removed net N$3: D1.A, DCC-2.KL, OK1.C
- new net DCC_1: B2.AC1, DCC-1.KL, R1.1
- new net DCC_2: B2.AC2, D1.A, DCC-2.KL, OK1.C
- new net N$10: Q1.E, R4.1
- new net N$11: B2.+, R4.2
- new net N$4: ACK.1, R3.1
- new net N$8: OK2.A, R3.2
- new net N$9: OK2.COL, Q1.B
- net GND: now also OK2.C
- net N$1: now also B2.-, OK2.EMIT, Q1.C; no longer DCC-1.KL, R1.1
Changed lines of the file:
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@@
 <?xml version="1.0" encoding="utf-8"?>
 <!DOCTYPE eagle SYSTEM "eagle.dtd">
-<eagle version="7.7.0">
+<eagle version="8.3.1">
 <drawing>
 <settings>
 <setting alwaysvectorfont="no"/>
+<setting keepoldvectorfont="yes"/>
 <setting verticaltext="up"/>
 </settings>
@@
 <part name="P+2" library="supply1" deviceset="+5V" device=""/>
 <part name="R2" library="rcl" deviceset="R-EU_" device="0207/10" value="10k"/>
+<part name="ACK" library="pinhead" library_urn="urn:adsk.eagle:library:325" deviceset="PINHD-1X1" device="" package3d_urn="urn:adsk.eagle:package:22485/1"/>
+<part name="OK2" library="optocoupler" library_urn="urn:adsk.eagle:library:320" deviceset="PC817" device="" package3d_urn="urn:adsk.eagle:package:21938/1"/>
+<part name="R3" library="rcl" deviceset="R-EU_" device="0207/10" value="1k"/>
+<part name="GND3" library="supply1" deviceset="GND" device=""/>
+<part name="B2" library="rectifier" library_urn="urn:adsk.eagle:library:336" deviceset="RB1A" device="" package3d_urn="urn:adsk.eagle:package:23866/1"/>
+<part name="Q1" library="transistor-pnp" library_urn="urn:adsk.eagle:library:399" deviceset="BC557" device="" package3d_urn="urn:adsk.eagle:package:29211/1"/>
+<part name="R4" library="rcl" deviceset="R-EU_" device="0207/10" value="100"/>
 </parts>
 <sheets>
@@
 <instance part="P+2" gate="1" x="68.58" y="58.42"/>
 <instance part="R2" gate="G$1" x="76.2" y="48.26"/>
+<instance part="ACK" gate="G$1" x="17.78" y="2.54"/>
+<instance part="OK2" gate="A" x="45.72" y="0"/>
+<instance part="R3" gate="G$1" x="27.94" y="2.54"/>
+<instance part="GND3" gate="1" x="33.02" y="-12.7"/>
+<instance part="B2" gate="1" x="78.74" y="-7.62"/>
+<instance part="Q1" gate="G$1" x="60.96" y="2.54"/>
+<instance part="R4" gate="G$1" x="73.66" y="10.16"/>
 </instances>
 <busses>
@@
 <wire x1="68.58" y1="40.64" x2="68.58" y2="38.1" width="0.1524" layer="91"/>
 </segment>
+<segment>
+<pinref part="OK2" gate="A" pin="C"/>
+<pinref part="GND3" gate="1" pin="GND"/>
+<wire x1="35.56" y1="-2.54" x2="33.02" y2="-2.54" width="0.1524" layer="91"/>
+<wire x1="33.02" y1="-2.54" x2="33.02" y2="-10.16" width="0.1524" layer="91"/>
+</segment>
 </net>
 <net name="+5V" class="0">
@@
 </segment>
 </net>
-<net name="N$1" class="0">
+<net name="DCC_1" class="0">
 <segment>
 <pinref part="DCC" gate="-1" pin="KL"/>
 <pinref part="R1" gate="G$1" pin="1"/>
 <wire x1="17.78" y1="48.26" x2="20.32" y2="48.26" width="0.1524" layer="91"/>
+</segment>
+<segment>
+<pinref part="B2" gate="1" pin="AC1"/>
+<wire x1="78.74" y1="-2.54" x2="78.74" y2="0" width="0.1524" layer="91"/>
+<wire x1="78.74" y1="0" x2="68.58" y2="0" width="0.1524" layer="91"/>
+<label x="68.58" y="0" size="1.778" layer="95"/>
 </segment>
 </net>
@@
 </segment>
 </net>
-<net name="N$3" class="0">
+<net name="DCC_2" class="0">
 <segment>
 <pinref part="DCC" gate="-2" pin="KL"/>
@@
 <junction x="35.56" y="38.1"/>
 </segment>
+<segment>
+<pinref part="B2" gate="1" pin="AC2"/>
+<wire x1="78.74" y1="-12.7" x2="78.74" y2="-15.24" width="0.1524" layer="91"/>
+<wire x1="78.74" y1="-15.24" x2="88.9" y2="-15.24" width="0.1524" layer="91"/>
+<label x="81.28" y="-15.24" size="1.778" layer="95"/>
+</segment>
 </net>
 <net name="N$5" class="0">
@@
 </segment>
 </net>
+<net name="N$4" class="0">
+<segment>
+<pinref part="ACK" gate="G$1" pin="1"/>
+<pinref part="R3" gate="G$1" pin="1"/>
+<wire x1="15.24" y1="2.54" x2="22.86" y2="2.54" width="0.1524" layer="91"/>
+</segment>
+</net>
+<net name="N$8" class="0">
+<segment>
+<pinref part="R3" gate="G$1" pin="2"/>
+<pinref part="OK2" gate="A" pin="A"/>
+<wire x1="33.02" y1="2.54" x2="35.56" y2="2.54" width="0.1524" layer="91"/>
+</segment>
+</net>
+<net name="N$9" class="0">
+<segment>
+<pinref part="OK2" gate="A" pin="COL"/>
+<pinref part="Q1" gate="G$1" pin="B"/>
+<wire x1="53.34" y1="2.54" x2="58.42" y2="2.54" width="0.1524" layer="91"/>
+</segment>
+</net>
+<net name="N$1" class="0">
+<segment>
+<pinref part="Q1" gate="G$1" pin="C"/>
+<wire x1="63.5" y1="-2.54" x2="63.5" y2="-7.62" width="0.1524" layer="91"/>
+<pinref part="B2" gate="1" pin="-"/>
+<wire x1="63.5" y1="-7.62" x2="73.66" y2="-7.62" width="0.1524" layer="91"/>
+<pinref part="OK2" gate="A" pin="EMIT"/>
+<wire x1="53.34" y1="-2.54" x2="58.42" y2="-2.54" width="0.1524" layer="91"/>
+<wire x1="58.42" y1="-2.54" x2="58.42" y2="-7.62" width="0.1524" layer="91"/>
+<wire x1="58.42" y1="-7.62" x2="63.5" y2="-7.62" width="0.1524" layer="91"/>
+<junction x="63.5" y="-7.62"/>
+</segment>
+</net>
+<net name="N$10" class="0">
+<segment>
+<pinref part="R4" gate="G$1" pin="1"/>
+<pinref part="Q1" gate="G$1" pin="E"/>
+<wire x1="68.58" y1="10.16" x2="63.5" y2="10.16" width="0.1524" layer="91"/>
+<wire x1="63.5" y1="10.16" x2="63.5" y2="7.62" width="0.1524" layer="91"/>
+</segment>
+</net>
+<net name="N$11" class="0">
+<segment>
+<pinref part="R4" gate="G$1" pin="2"/>
+<wire x1="78.74" y1="10.16" x2="88.9" y2="10.16" width="0.1524" layer="91"/>
+<wire x1="88.9" y1="10.16" x2="88.9" y2="-7.62" width="0.1524" layer="91"/>
+<pinref part="B2" gate="1" pin="+"/>
+<wire x1="88.9" y1="-7.62" x2="83.82" y2="-7.62" width="0.1524" layer="91"/>
+</segment>
+</net>
 </nets>
 </sheet>
@@
 </schematic>
 </drawing>
+<compatibility>
+<note version="8.2" severity="warning">
+Since Version 8.2, EAGLE supports online libraries. The ids
+of those online libraries will not be understood (or retained)
+with this version.
+</note>
+<note version="8.3" severity="warning">
+Since Version 8.3, EAGLE supports URNs for individual library
+assets (packages, symbols, and devices). The URNs of those assets
+will not be understood (or retained) with this version.
+</note>
+<note version="8.3" severity="warning">
+Since Version 8.3, EAGLE supports the association of 3D packages
+with devices in libraries, schematics, and board files. Those 3D
+packages will not be understood (or retained) with this version.
+</note>
+</compatibility>
 </eagle>
